File: hardware/LM75-tryout.kicad_pcb (KiCad board)
At the start: 2 copper layers, 4 parts, among them J1 LM75_HEADER, U1 LM75

Commit message: update,
Parts:
- added JP1: EN, Jumper:SolderJumper-2_P1.3mm_Open_RoundedPad1.0x1.5mm, F.Cu at (23.0, 16.0)
Connections:
- C1 pad 1: +3V3 -> Net-(C1-Pad1)
- RN1 pad 6: +3V3 -> Net-(C1-Pad1)
- RN1 pad 7: +3V3 -> Net-(C1-Pad1)
- RN1 pad 8: +3V3 -> Net-(C1-Pad1)
- U1 pad 8: +3V3 -> Net-(C1-Pad1)
Routing:
- net Net-(C1-Pad1): track 0.00 -> 16.8 mm
- net +3V3: track 19.6 -> 15.8 mm
Changed lines of the file:
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@@
     (thickness 1.6)
     (drawings 0)
-    (tracks 54)
+    (tracks 58)
     (zones 0)
-    (modules 4)
-    (nets 6)
+    (modules 5)
+    (nets 7)
   )
   (page A4)
@@
   (net 4 "Net-(J1-Pad5)")
   (net 5 "Net-(J1-Pad4)")
+  (net 6 "Net-(C1-Pad1)")
   (net_class Default "This is the default net class."
     (clearance 0.2)
@@
     (add_net +3V3)
     (add_net GND)
+    (add_net "Net-(C1-Pad1)")
     (add_net "Net-(J1-Pad3)")
     (add_net "Net-(J1-Pad4)")
     (add_net "Net-(J1-Pad5)")
+    (add_net "Net-(RN1-Pad4)")
+    (add_net "Net-(RN1-Pad5)")
+  )
+  (module Jumper:SolderJumper-2_P1.3mm_Open_RoundedPad1.0x1.5mm (layer F.Cu)
+    (at 23 16)
+    (descr "SMD Solder Jumper, 1x1.5mm, rounded Pads, 0.3mm gap, open")
+    (tags "solder jumper open")
+    (attr virtual)
+    (fp_text reference JP1 (at 0 -1.8) (layer F.SilkS)
+      (effects (font (size 1 1) (thickness 0.15)))
+    )
+    (fp_text value EN (at 0 1.9) (layer F.Fab)
+      (effects (font (size 1 1) (thickness 0.15)))
+    )
+    (fp_line (start 1.65 1.25) (end -1.65 1.25) (layer F.CrtYd) (width 0.05))
+    (fp_line (start 1.65 1.25) (end 1.65 -1.25) (layer F.CrtYd) (width 0.05))
+    (fp_line (start -1.65 -1.25) (end -1.65 1.25) (layer F.CrtYd) (width 0.05))
+    (fp_line (start -1.65 -1.25) (end 1.65 -1.25) (layer F.CrtYd) (width 0.05))
+    (fp_line (start -0.7 -1) (end 0.7 -1) (layer F.SilkS) (width 0.12))
+    (fp_line (start 1.4 -0.3) (end 1.4 0.3) (layer F.SilkS) (width 0.12))
+    (fp_line (start 0.7 1) (end -0.7 1) (layer F.SilkS) (width 0.12))
+    (fp_line (start -1.4 0.3) (end -1.4 -0.3) (layer F.SilkS) (width 0.12))
+    (fp_arc (start -0.7 -0.3) (end -0.7 -1) (angle -90) (layer F.SilkS) (width 0.12))
+    (fp_arc (start -0.7 0.3) (end -1.4 0.3) (angle -90) (layer F.SilkS) (width 0.12))
+    (fp_arc (start 0.7 0.3) (end 0.7 1) (angle -90) (layer F.SilkS) (width 0.12))
+    (fp_arc (start 0.7 -0.3) (end 1.4 -0.3) (angle -90) (layer F.SilkS) (width 0.12))
+    (pad 2 smd custom (at 0.65 0) (size 1 0.5) (layers F.Cu F.Mask)
+      (net 6 "Net-(C1-Pad1)") (zone_connect 2)
+      (options (clearance outline) (anchor rect))
+      (primitives
+        (gr_circle (center 0 0.25) (end 0.5 0.25) (width 0))
+        (gr_circle (center 0 -0.25) (end 0.5 -0.25) (width 0))
+        (gr_poly (pts
+           (xy 0 -0.75) (xy -0.5 -0.75) (xy -0.5 0.75) (xy 0 0.75)) (width 0))
+      ))
+    (pad 1 smd custom (at -0.65 0) (size 1 0.5) (layers F.Cu F.Mask)
+      (net 2 +3V3) (zone_connect 2)
+      (options (clearance outline) (anchor rect))
+      (primitives
+        (gr_circle (center 0 0.25) (end 0.5 0.25) (width 0))
+        (gr_circle (center 0 -0.25) (end 0.5 -0.25) (width 0))
+        (gr_poly (pts
+           (xy 0 -0.75) (xy 0.5 -0.75) (xy 0.5 0.75) (xy 0 0.75)) (width 0))
+      ))
   )
   (module Connector_PinHeader_1.27mm:PinHeader_1x05_P1.27mm_Vertical (layer F.Cu)
@@
     (fp_line (start 0 2.59) (end 1.88 2.59) (layer F.SilkS) (width 0.12))
     (pad 8 smd roundrect (at 2.5375 -1.905) (size 1.975 0.65) (layers F.Cu F.Paste F.Mask) (roundrect_rratio 0.25)
-      (net 2 +3V3))
+      (net 6 "Net-(C1-Pad1)"))
     (pad 7 smd roundrect (at 2.5375 -0.635) (size 1.975 0.65) (layers F.Cu F.Paste F.Mask) (roundrect_rratio 0.25)
       (net 1 GND))
@@
     (pad 5 smd rect (at 0.85 1.2 90) (size 0.9 0.4) (layers F.Cu F.Paste F.Mask))
     (pad 6 smd rect (at 0.85 0.4 90) (size 0.9 0.4) (layers F.Cu F.Paste F.Mask)
-      (net 2 +3V3))
+      (net 6 "Net-(C1-Pad1)"))
     (pad 7 smd rect (at 0.85 -0.4 90) (size 0.9 0.4) (layers F.Cu F.Paste F.Mask)
-      (net 2 +3V3))
+      (net 6 "Net-(C1-Pad1)"))
     (pad 8 smd rect (at 0.85 -1.2 90) (size 0.9 0.4) (layers F.Cu F.Paste F.Mask)
-      (net 2 +3V3))
+      (net 6 "Net-(C1-Pad1)"))
     (pad 4 smd rect (at -0.85 1.2 90) (size 0.9 0.4) (layers F.Cu F.Paste F.Mask))
     (pad 1 smd rect (at -0.85 -1.2 90) (size 0.9 0.4) (layers F.Cu F.Paste F.Mask)
@@
       (net 1 GND))
     (pad 1 smd roundrect (at -0.875 0 180) (size 1.05 0.95) (layers F.Cu F.Paste F.Mask) (roundrect_rratio 0.25)
-      (net 2 +3V3))
+      (net 6 "Net-(C1-Pad1)"))
     (model ${KISYS3DMOD}/Capacitor_SMD.3dshapes/C_0603_1608Metric.wrl
       (at (xyz 0 0 0))
@@
   (segment (start 22.125 20.7922) (end 23.1878 21.855) (width 0.25) (layer F.Cu) (net 1))
   (segment (start 23.1878 21.855) (end 23.6675 21.855) (width 0.25) (layer F.Cu) (net 1))
-  (segment (start 13.8 17.0343) (end 12.7 18.1343) (width 0.25) (layer F.Cu) (net 2))
-  (segment (start 12.7 18.1343) (end 12.7 21.2) (width 0.25) (layer F.Cu) (net 2))
-  (segment (start 13.8 17.0343) (end 13.8 16.9186) (width 0.25) (layer F.Cu) (net 2))
-  (segment (start 13.8 17.15) (end 13.8 17.0343) (width 0.25) (layer F.Cu) (net 2))
-  (segment (start 14.6 16.9561) (end 14.5626 16.9187) (width 0.25) (layer F.Cu) (net 2))
-  (segment (start 14.5626 16.9187) (end 14.5626 16.9186) (width 0.25) (layer F.Cu) (net 2))
-  (segment (start 14.5626 16.9186) (end 13.8 16.9186) (width 0.25) (layer F.Cu) (net 2))
-  (segment (start 14.6 16.9561) (end 14.6 16.7623) (width 0.25) (layer F.Cu) (net 2))
-  (segment (start 14.6 17.15) (end 14.6 16.9561) (width 0.25) (layer F.Cu) (net 2))
-  (segment (start 15.4 16.3747) (end 14.9876 16.3747) (width 0.25) (layer F.Cu) (net 2))
-  (segment (start 14.9876 16.3747) (end 14.6 16.7623) (width 0.25) (layer F.Cu) (net 2))
-  (segment (start 23.875 18) (end 22.2497 16.3747) (width 0.25) (layer F.Cu) (net 2))
-  (segment (start 22.2497 16.3747) (end 15.4 16.3747) (width 0.25) (layer F.Cu) (net 2))
-  (segment (start 23.6675 20.585) (end 23.875 20.3775) (width 0.25) (layer F.Cu) (net 2))
-  (segment (start 23.875 20.3775) (end 23.875 18) (width 0.25) (layer F.Cu) (net 2))
-  (segment (start 15.4 17.15) (end 15.4 16.3747) (width 0.25) (layer F.Cu) (net 2))
+  (segment (start 18.036401 15.749991) (end 13.100009 15.749991) (width 0.25) (layer F.Cu) (net 2))
+  (segment (start 22.35 16) (end 18.28641 16) (width 0.25) (layer F.Cu) (net 2))
+  (segment (start 18.28641 16) (end 18.036401 15.749991) (width 0.25) (layer F.Cu) (net 2))
+  (segment (start 12.7 16.15) (end 12.7 19) (width 0.25) (layer F.Cu) (net 2))
+  (segment (start 13.100009 15.749991) (end 12.7 16.15) (width 0.25) (layer F.Cu) (net 2))
+  (segment (start 12.7 18.1343) (end 12.7 19) (width 0.25) (layer F.Cu) (net 2))
+  (segment (start 12.7 19) (end 12.7 21.2) (width 0.25) (layer F.Cu) (net 2))
+  (segment (start 13.8 17.15) (end 13.8 17.0343) (width 0.25) (layer F.Cu) (net 6))
+  (segment (start 23.6675 20.585) (end 23.875 20.3775) (width 0.25) (layer F.Cu) (net 6))
+  (segment (start 23.875 20.3775) (end 23.875 18) (width 0.25) (layer F.Cu) (net 6))
   (segment (start 13.8 20.585) (end 13.8 22.64) (width 0.25) (layer F.Cu) (net 3))
   (segment (start 13.8 22.64) (end 12.7 23.74) (width 0.25) (layer F.Cu) (net 3))
@@
   (segment (start 16.6803 21.855) (end 18.5925 21.855) (width 0.25) (layer F.Cu) (net 5))
   (segment (start 12.7 25.01) (end 13.5253 25.01) (width 0.25) (layer F.Cu) (net 5))
+  (segment (start 23.875 16.225) (end 23.65 16) (width 0.25) (layer F.Cu) (net 6))
+  (segment (start 23.875 18) (end 23.875 16.225) (width 0.25) (layer F.Cu) (net 6))
+  (segment (start 23.65 16) (end 23.65 16.847592) (width 0.25) (layer F.Cu) (net 6))
+  (segment (start 23.422582 17.07501) (end 18.72501 17.07501) (width 0.25) (layer F.Cu) (net 6))
+  (segment (start 23.65 16.847592) (end 23.422582 17.07501) (width 0.25) (layer F.Cu) (net 6))
+  (segment (start 18.72501 17.07501) (end 17.85 16.2) (width 0.25) (layer F.Cu) (net 6))
+  (segment (start 15.65 16.2) (end 15.4 16.45) (width 0.25) (layer F.Cu) (net 6))
+  (segment (start 15.4 16.45) (end 15.4 17.15) (width 0.25) (layer F.Cu) (net 6))
+  (segment (start 17.85 16.2) (end 15.65 16.2) (width 0.25) (layer F.Cu) (net 6))
+  (segment (start 15.4 17.15) (end 13.8 17.15) (width 0.25) (layer F.Cu) (net 6))
 )
